File: PCB/Fan-Module.brd (EAGLE design)
At the start: 58 x 66 mm, 28 parts, among them U1 ATSAMD11C14A-SSUT_ATSAMD11C14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, U3 LDL1117S12R_LDL1117S12R

Commit message: added 4pin connector for remaining pins on all boards
Parts:
- added J3: (no value), SparkFun-Connectors:1X04
- moved J2 10.5 mm to (57.9, 10.2), turned to 90 degrees
Connections:
- new net N$10: J3.2, U1.3
- new net N$11: J3.1, U1.4
- new net N$7: J3.4, U1.1
- new net N$9: J3.3, U1.2
Routing:
- net N$10: track 0.00 -> 40.1 mm, vias 0 -> 2
- net N$11: track 0.00 -> 32.7 mm, vias 0 -> 2
- net N$7: track 0.00 -> 32.6 mm
- net N$9: track 0.00 -> 32.4 mm
- net GND: track 22.8 -> 28.7 mm
- net 3.3V: track 68.3 -> 63.4 mm
- net RESET: track 33.2 -> 28.9 mm
- net SWDIO: track 34.5 -> 31.2 mm, vias 1 -> 0
- net SWCLK: track 29.4 -> 27.1 mm
- net N$5: track 53.6 -> 51.5 mm, vias 0 -> 2
- net N$3: track 34.6 -> 35.1 mm, vias 0 -> 2
