File: PCB/LED-Board.brd (EAGLE design)
At the start: 71 x 34 mm, 33 parts, among them U1 ATSAMD11C14A-SSUT, U3 LDL1117S12R

Commit message: added 4pin connector for remaining pins on all boards
Changed lines of the file:
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@@
 </element>
 <element name="C6" library="microbuilder" package="0603" value="1uF" x="49.5656" y="11.0532" smashed="yes">
-<attribute name="NAME" x="51.3436" y="10.9262" size="0.762" layer="25" font="vector" ratio="15"/>
-<attribute name="VALUE" x="51.3436" y="10.2912" size="0.4064" layer="27" font="vector" ratio="10"/>
+<attribute name="NAME" x="49.9436" y="11.9262" size="0.762" layer="25" font="vector" ratio="15"/>
+<attribute name="VALUE" x="50.0436" y="9.6912" size="0.4064" layer="27" font="vector" ratio="10"/>
 </element>
 <element name="U1" library="ATSAMD11C14A-SSUT" package="SOIC127P600X160-14N" value="ATSAMD11C14A-SSUT" x="49.61" y="5.1952" smashed="yes" rot="R90">
