File: PCB/Fan-Module_80mm.brd (EAGLE design)
At the start: 83 x 97 mm, 31 parts, among them U1 ATSAMD11C14A-SSUT_ATSAMD11C14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, U3 LDL1117S12R_LDL1117S12R

Commit message: unknown changes, break has been too long
Parts:
- moved D3 0.92 mm to (12.9, 83.4)
- moved D1 0.67 mm to (16.2, 83.4)
Routing:
- net GND: track 267.5 -> 265.4 mm
- net SWDIO: track 28.7 -> 27.8 mm
- net N$4: track 61.9 -> 61.1 mm
- net RESET: track 23.2 -> 23.8 mm
