File: PCB/water-pump.brd (EAGLE design)
At the start: 53 x 66.3 mm, 27 parts, among them U1 LDL1117S12R, U3 ATSAMD11C14A-SSUT

Commit message: added 4pin connector for remaining pins on all boards
Parts:
- added J3: (no value), SparkFun-Connectors:1X04
- moved J2 6.26 mm to (47.0, 13.3)
Connections:
- new net N$10: J3.2, U3.3
- new net N$11: J3.1, U3.4
- new net N$4: J3.4, U3.1
- new net N$9: J3.3, U3.2
Routing:
- net N$4: track 0.00 -> 51.8 mm
- net N$9: track 0.00 -> 47.1 mm
- net N$10: track 0.00 -> 42.5 mm
- net N$11: track 0.00 -> 36.6 mm
- net SWCLK: track 33.0 -> 29.1 mm
- net RESET: track 34.2 -> 30.2 mm
- net 3.3V: track 80.4 -> 78.8 mm
- net SWDIO: track 30.0 -> 29.5 mm
- net N$3: track 18.4 -> 18.5 mm, vias 0 -> 2
Changed lines of the file:
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@@
 <?xml version="1.0" encoding="utf-8"?>
 <!DOCTYPE eagle SYSTEM "eagle.dtd">
-<eagle version="9.3.0">
+<eagle version="9.2.2">
 <drawing>
 <settings>
-<setting alwaysvectorfont="yes"/>
+<setting alwaysvectorfont="no"/>
 <setting keepoldvectorfont="yes"/>
 <setting verticaltext="up"/>
@@
 <attribute name="VALUE" x="8.679" y="18.87" size="1.27" layer="27" rot="R90"/>
 </element>
-<element name="J2" library="SparkFun-Connectors" package="1X05" value="" x="48.4" y="7.203" smashed="yes" rot="R90">
-<attribute name="NAME" x="47.003" y="5.933" size="0.762" layer="25" font="vector" ratio="15" rot="R90"/>
-<attribute name="VALUE" x="50.432" y="5.933" size="0.6096" layer="27" font="vector" ratio="20" rot="R90"/>
+<element name="J2" library="SparkFun-Connectors" package="1X05" value="" x="47" y="13.303" smashed="yes" rot="R90">
+<attribute name="NAME" x="47.303" y="10.533" size="0.762" layer="25" font="vector" ratio="15" rot="R90"/>
+<attribute name="VALUE" x="49.032" y="12.033" size="0.6096" layer="27" font="vector" ratio="20" rot="R90"/>
 </element>
 <element name="D3" library="SparkFun-DiscreteSemi" package="SMA-DIODE" value="3A/40V/500mV" x="3.907" y="20.625" smashed="yes" rot="MR90">
@@
 <attribute name="NAME" x="24.343" y="20.83" size="0.4064" layer="26" rot="MR90"/>
 <attribute name="VALUE" x="24.376" y="18.403" size="0.4064" layer="28" rot="MR90"/>
+</element>
+<element name="J3" library="SparkFun-Connectors" package="1X04" value="" x="49.6" y="23.4" smashed="yes" rot="R270">
+<attribute name="NAME" x="49.297" y="25.97" size="0.6096" layer="25" font="vector" ratio="20" rot="R270"/>
+<attribute name="PROD_ID" value="CONN-09696" x="49.6" y="23.4" size="1.778" layer="27" rot="R270" display="off"/>
+<attribute name="VALUE" x="47.568" y="24.67" size="0.6096" layer="27" font="vector" ratio="20" rot="R270"/>
 </element>
 </elements>
@@
 <contactref element="R1" pad="2"/>
 <contactref element="U3" pad="5"/>
-<wire x1="17.475" y1="21.139" x2="17.475" y2="28.91" width="0.6096" layer="16"/>
 <wire x1="17.475" y1="28.91" x2="24.993" y2="36.428" width="0.6096" layer="16"/>
+<wire x1="17.475" y1="21.139" x2="17.475" y2="23.3" width="0.6096" layer="16"/>
+<wire x1="17.475" y1="23.3" x2="17.5" y2="23.3" width="0.6096" layer="16"/>
+<via x="17.5" y="23.3" extent="1-16" drill="0.3937"/>
+<via x="17.5" y="28.2" extent="1-16" drill="0.3937"/>
+<wire x1="17.5" y1="28.2" x2="17.5" y2="28.91" width="0.6096" layer="16"/>
+<wire x1="17.5" y1="28.91" x2="17.475" y2="28.91" width="0.6096" layer="16"/>
+<wire x1="17.5" y1="23.3" x2="17.5" y2="28.2" width="0.6096" layer="1"/>
 </signal>
 <signal name="N$7">
@@
 <wire x1="21.954" y1="14.3" x2="22.6" y2="14.3" width="0.3048" layer="16"/>
 <via x="22.6" y="14.3" extent="1-16" drill="0.55"/>
-<wire x1="22.6" y1="14.3" x2="46.383" y2="14.3" width="0.3048" layer="1"/>
-<wire x1="46.383" y1="14.3" x2="48.4" y2="12.283" width="0.3048" layer="1"/>
+<wire x1="22.6" y1="14.3" x2="42.917" y2="14.3" width="0.3048" layer="1"/>
+<wire x1="42.917" y1="14.3" x2="47" y2="18.383" width="0.3048" layer="1"/>
 </signal>
 <signal name="SWCLK">
@@
 <contactref element="J2" pad="4"/>
 <wire x1="20.015" y1="21.139" x2="20.015" y2="22.315" width="0.3048" layer="16"/>
-<wire x1="40.523" y1="22.7" x2="48.4" y2="14.823" width="0.3048" layer="16"/>
+<wire x1="45.223" y1="22.7" x2="47" y2="20.923" width="0.3048" layer="16"/>
 <wire x1="20.015" y1="22.315" x2="20.4" y2="22.7" width="0.3048" layer="16"/>
-<wire x1="20.4" y1="22.7" x2="40.523" y2="22.7" width="0.3048" layer="16"/>
+<wire x1="20.4" y1="22.7" x2="45.223" y2="22.7" width="0.3048" layer="16"/>
 </signal>
 <signal name="N$1">
@@
 <wire x1="18.745" y1="21.139" x2="18.745" y2="22.845" width="0.3048" layer="16"/>
 <wire x1="18.745" y1="22.845" x2="19.4" y2="23.5" width="0.3048" layer="16"/>
-<wire x1="19.4" y1="23.5" x2="42.263" y2="23.5" width="0.3048" layer="16"/>
-<wire x1="42.263" y1="23.5" x2="48.4" y2="17.363" width="0.3048" layer="16"/>
+<wire x1="19.4" y1="23.5" x2="46.963" y2="23.5" width="0.3048" layer="16"/>
+<wire x1="46.963" y1="23.5" x2="47" y2="23.463" width="0.3048" layer="16"/>
 </signal>
 <signal name="N$6" class="1">
@@
 <wire x1="10.3" y1="19.3" x2="7.90894375" y2="19.3" width="0.3048" layer="1"/>
 <wire x1="7.90894375" y1="19.3" x2="7.36654375" y2="19.8424" width="0.3048" layer="1"/>
-<wire x1="48.4" y1="9.743" x2="45.143" y2="13" width="0.3048" layer="1"/>
+<wire x1="47" y1="15.843" x2="44.157" y2="13" width="0.3048" layer="1"/>
 <wire x1="15.58080625" y1="14.31919375" x2="16.9" y2="13" width="0.3048" layer="1"/>
 <via x="15.58080625" y="14.31919375" extent="1-16" drill="0.55"/>
 <wire x1="15.58080625" y1="14.31919375" x2="14.935" y2="14.965" width="0.3048" layer="16"/>
 <wire x1="14.935" y1="14.965" x2="14.935" y2="16" width="0.3048" layer="16"/>
-<wire x1="45.143" y1="13" x2="24" y2="13" width="0.3048" layer="1"/>
+<wire x1="44.157" y1="13" x2="24" y2="13" width="0.3048" layer="1"/>
 <wire x1="18.3" y1="13" x2="18.3015875" y2="12.9984125" width="0.3048" layer="1"/>
 <via x="18.3015875" y="12.9984125" extent="1-16" drill="0.55"/>
@@
 <wire x1="29" y1="20.9" x2="30.625" y2="20.9" width="0.6096" layer="16"/>
 </signal>
+<signal name="N$4">
+<contactref element="U3" pad="1"/>
+<contactref element="J3" pad="4"/>
+<wire x1="12.423615625" y1="21.167615625" x2="12.395" y2="21.139" width="0.2032" layer="16"/>
+<wire x1="12.4" y1="21.144" x2="12.395" y2="21.139" width="0.2032" layer="16"/>
+<wire x1="49.6" y1="15.78" x2="49.6" y2="16.52394375" width="0.254" layer="16"/>
+<wire x1="49.6" y1="16.52394375" x2="51.7844" y2="18.70834375" width="0.254" layer="16"/>
+<wire x1="51.7844" y1="24.30481875" x2="51.7844" y2="18.70834375" width="0.254" layer="16"/>
+<wire x1="13.0348" y1="22.1000375" x2="13.0348" y2="21.7788" width="0.254" layer="16"/>
+<wire x1="13.0348" y1="21.7788" x2="12.423615625" y2="21.167615625" width="0.254" layer="16"/>
+<wire x1="17.0393625" y1="26.1046" x2="49.98461875" y2="26.1046" width="0.254" layer="16"/>
+<wire x1="17.0393625" y1="26.1046" x2="13.0348" y2="22.1000375" width="0.254" layer="16"/>
+<wire x1="49.98461875" y1="26.1046" x2="51.7844" y2="24.30481875" width="0.254" layer="16"/>
+</signal>
+<signal name="N$9">
+<contactref element="U3" pad="2"/>
+<contactref element="J3" pad="3"/>
+<wire x1="13.6" y1="21.204" x2="13.602" y2="21.202" width="0.2032" layer="16"/>
+<wire x1="13.602" y1="21.202" x2="13.665" y2="21.139" width="0.2032" layer="16"/>
+<wire x1="13.7" y1="21.3" x2="13.602" y2="21.202" width="0.2032" layer="16"/>
+<wire x1="51.3272" y1="24.1154375" x2="49.7952375" y2="25.6474" width="0.254" layer="16"/>
+<wire x1="51.3272" y1="20.79114375" x2="51.3272" y2="24.1154375" width="0.254" layer="16"/>
+<wire x1="49.6" y1="18.32" x2="49.6" y2="19.06394375" width="0.254" layer="16"/>
+<wire x1="49.6" y1="19.06394375" x2="51.3272" y2="20.79114375" width="0.254" layer="16"/>
+<wire x1="14.3048" y1="21.9048" x2="13.7" y2="21.3" width="0.254" layer="16"/>
+<wire x1="17.52150625" y1="25.6474" x2="14.3048" y2="22.43069375" width="0.254" layer="16"/>
+<wire x1="14.3048" y1="22.43069375" x2="14.3048" y2="21.9048" width="0.254" layer="16"/>
+<wire x1="49.7952375" y1="25.6474" x2="17.52150625" y2="25.6474" width="0.254" layer="16"/>
+</signal>
+<signal name="N$10">
+<contactref element="U3" pad="3"/>
+<contactref element="J3" pad="2"/>
+<wire x1="50.87" y1="22.87394375" x2="50.87" y2="23.92605625" width="0.254" layer="16"/>
+<wire x1="50.87" y1="23.92605625" x2="49.60585625" y2="25.1902" width="0.254" layer="16"/>
+<wire x1="49.6" y1="20.86" x2="49.6" y2="21.60394375" width="0.254" layer="16"/>
+<wire x1="49.6" y1="21.60394375" x2="50.87" y2="22.87394375" width="0.254" layer="16"/>
+<wire x1="15.5748" y1="21.7788" x2="14.935" y2="21.139" width="0.254" layer="16"/>
+<wire x1="17.7108875" y1="25.1902" x2="15.5748" y2="23.0541125" width="0.254" layer="16"/>
+<wire x1="15.5748" y1="23.0541125" x2="15.5748" y2="21.7788" width="0.254" layer="16"/>
+<wire x1="49.60585625" y1="25.1902" x2="17.7108875" y2="25.1902" width="0.254" layer="16"/>
+</signal>
+<signal name="N$11">
+<contactref element="U3" pad="4"/>
+<contactref element="J3" pad="1"/>
+<wire x1="49.6" y1="23.4" x2="48.85905625" y2="23.4" width="0.254" layer="16"/>
+<wire x1="16.76975" y1="23.60248125" x2="16.76975" y2="23.56975" width="0.254" layer="16"/>
+<wire x1="48.85905625" y1="23.4" x2="47.52605625" y2="24.733" width="0.254" layer="16"/>
+<wire x1="47.52605625" y1="24.733" x2="17.90026875" y2="24.733" width="0.254" layer="16"/>
+<wire x1="17.90026875" y1="24.733" x2="16.76975" y2="23.60248125" width="0.254" layer="16"/>
+<wire x1="16.76975" y1="23.56975" x2="16.2" y2="23" width="0.254" layer="16"/>
+<wire x1="16.2" y1="23" x2="16.205" y2="22.995" width="0.254" layer="16"/>
+<wire x1="16.205" y1="22.995" x2="16.205" y2="21.139" width="0.254" layer="16"/>
+</signal>
 </signals>

Commit message: unknown changes, break has been too long
Parts:
- moved J10 6.41 mm to (31.1, 5.96)
Routing:
- net VCC: track 63.9 -> 69.8 mm
- net PUMP: track 13.3 -> 14.1 mm
- net N$1: track 7.21 -> 7.75 mm
Changed lines of the file:
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@@
 <?xml version="1.0" encoding="utf-8"?>
 <!DOCTYPE eagle SYSTEM "eagle.dtd">
-<eagle version="9.2.2">
+<eagle version="9.3.0">
 <drawing>
 <settings>
@@
 <attribute name="VALUE" x="0.704" y="5.925" size="0.6096" layer="27" font="vector" ratio="20" align="top-left"/>
 </element>
-<element name="J10" library="SparkFun-Connectors" library_urn="urn:adsk.eagle:library:513" package="1X02_LONGPADS" package3d_urn="urn:adsk.eagle:package:38048/1" value="" x="24.694" y="6.362" smashed="yes">
-<attribute name="NAME" x="24.624" y="8.494" size="0.762" layer="25" font="vector" ratio="15"/>
-<attribute name="VALUE" x="23.297" y="3.695" size="0.6096" layer="27" font="vector" ratio="20"/>
+<element name="J10" library="SparkFun-Connectors" library_urn="urn:adsk.eagle:library:513" package="1X02_LONGPADS" package3d_urn="urn:adsk.eagle:package:38048/1" value="" x="31.094" y="5.962" smashed="yes">
+<attribute name="NAME" x="31.024" y="8.094" size="0.762" layer="25" font="vector" ratio="15"/>
+<attribute name="VALUE" x="29.697" y="3.295" size="0.6096" layer="27" font="vector" ratio="20"/>
 </element>
 <element name="U3" library="ATSAMD11C14A-SSUT" package="SOIC127P600X160-14N" value="ATSAMD11C14A-SSUT" x="16.205" y="18.689" smashed="yes" rot="MR270">
@@
 <wire x1="3.907" y1="23.275" x2="3.907" y2="22.775" width="0.6096" layer="16"/>
 <wire x1="3.9" y1="36.4" x2="7.9" y2="32.4" width="0.6096" layer="16"/>
-<wire x1="24.694" y1="6.362" x2="20.8" y2="10.256" width="0.6096" layer="16"/>
-<wire x1="20.8" y1="10.256" x2="20.8" y2="11.3" width="0.6096" layer="16"/>
+<wire x1="31.094" y1="5.962" x2="30.994" y2="5.962" width="0.6096" layer="16"/>
+<wire x1="30.994" y1="5.962" x2="30.956" y2="6" width="0.6096" layer="16"/>
+<wire x1="30.956" y1="6" x2="26.1" y2="6" width="0.6096" layer="16"/>
+<wire x1="20.8" y1="11.3" x2="26.1" y2="6" width="0.6096" layer="16"/>
 <via x="20.8" y="11.3" extent="1-16" drill="0.55"/>
 <via x="7.832" y="27.2" extent="1-16" drill="0.55"/>
@@
 <contactref element="J10" pad="2"/>
 <contactref element="Q1" pad="3"/>
-<wire x1="30.034" y1="18.541" x2="30.034" y2="9.162" width="0.6096" layer="16"/>
-<wire x1="30.034" y1="9.162" x2="27.234" y2="6.362" width="0.6096" layer="16"/>
+<wire x1="30.034" y1="18.541" x2="30.034" y2="11.762" width="0.6096" layer="16"/>
+<wire x1="33.634" y1="8.162" x2="33.634" y2="5.962" width="0.6096" layer="16"/>
+<wire x1="33.634" y1="8.162" x2="30.034" y2="11.762" width="0.6096" layer="16"/>
 </signal>
 <signal name="USB+">
@@
 <contactref element="J1" pad="VBUS"/>
 <contactref element="D3" pad="A"/>
-<wire x1="4.699" y1="11.924" x2="5.1" y2="12.325" width="0.4064" layer="1"/>
-<wire x1="5.1" y1="12.325" x2="5.1" y2="17.2" width="0.4064" layer="1"/>
+<wire x1="5.4" y1="12.125" x2="5.199" y2="11.924" width="0.4064" layer="1"/>
+<wire x1="4.699" y1="11.924" x2="5.199" y2="11.924" width="0.4064" layer="1"/>
+<wire x1="5.4" y1="16.9" x2="5.1" y2="17.2" width="0.4064" layer="1"/>
+<wire x1="5.4" y1="16.9" x2="5.4" y2="12.125" width="0.4064" layer="1"/>
 <via x="5.1" y="17.2" extent="1-16" drill="0.55"/>
 <wire x1="5.1" y1="17.2" x2="5.1" y2="17.282" width="0.4064" layer="16"/>
